File: schematic/03_io_and_telemetry.kicad_sch (KiCad schematic)
At the start: 33 parts, among them Q301 DMN62D2UQ-7, Q302 DMN62D2UQ-7, U301 TPS62131RGTR, U302 INA226 0x40, U303 INA226 0x41, U509 TLV3011AIDBVR

Commit message: Decouple DUT reset and input diagnostics from power interlocks
Use explicit manual, ZedBoard, and Pico reset requests. Route input-voltage validity to telemetry while retaining protective power interlocks. Synchronize requirements, schematic exports, BOM, and verification evidence.
Parts:
- added R516: 10k / 1%, Sphinx_V2:Resistor_SMD__R_0603_1608Metric, symbol Sphinx_V2:Device__R
Connections:
- net 3V3_CTRL: now also R516.1
- net HW_FAULT_N renamed VIN12_VALID
- net VIN12_VALID: now also R516.2
Other:
- note added: "FSW tied to PG selects about 1.25MHz after startup. PG may float HIGH while OFF; U508 IO_VALID monitors VIO independently."
- note added: "U509: VIN12_VALID to Pico GP12, monitor-only; nominal threshold10.33V. Intrinsic UVLO or control brownout can still interrupt rails."
- note removed: "FSW tied to PG selects about 1.25MHz after startup. PG may float HIGH while OFF: reset uses independent U508 IO_VALID."
- note removed: "U509: VIN12 loss clears RUN_LATCH. Nominal trip10.33V; qualify fast input interruptions with USB connected."
Changed lines of the file:
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@@
 (kicad_sch (version 20250114) (generator "eeschema") (generator_version "10.0")
  (paper "A3")
-        (title_block (title "03 | Fixed 1.8 V I/O and calibrated telemetry") (date "2026-09-19") (rev "V2")
+        (title_block (title "03 | Fixed 1.8 V I/O and calibrated telemetry") (date "2026-09-20") (rev "V2")
         (company "Sphinx | Programmable power test board")
         (comment 1 "Review package: PCB, PI, SI, thermal and ASIC limits require qualification")
@@
 (wire (pts (xy 369.57 125.73) (xy 369.57 130.81)) (stroke (width 0) (type default)))
 (global_label "GND" (shape passive) (at 369.57 130.81 180) (effects (font (size 1.0 1.0)) (justify right) ) (property "Intersheetrefs" "${INTERSHEET_REFS}" (at 369.57 130.81 180) (effects (font (size 0.8 0.8))  (hide yes))))
-(text "FSW tied to PG selects about 1.25MHz after startup. PG may float HIGH while OFF: reset uses independent U508 IO_VALID." (at 15 167 0) (effects (font (size 0.98 0.98)) (justify left top) ))
+(text "FSW tied to PG selects about 1.25MHz after startup. PG may float HIGH while OFF; U508 IO_VALID monitors VIO independently." (at 15 167 0) (effects (font (size 0.98 0.98)) (justify left top) ))
 (symbol (lib_id "Sphinx_V2:INA226") (at 69.85 219.71 0) (unit 1) (exclude_from_sim no) (in_bom yes) (on_board yes) (dnp no)
 (property "Reference" "U302" (at 69.85 193.39 0) (effects (font (size 1.0 1.0))  ))
@@
 (property "Datasheet" "https://www.ti.com/lit/ds/symlink/tlv3011.pdf" (at 340.36 219.71 0) (effects (font (size 1.0 1.0))  (hide yes)))
 (property "MPN" "TLV3011AIDBVR" (at 340.36 219.71 0) (effects (font (size 1.0 1.0))  (hide yes)))
-(property "Description" "Post-eFuse VIN12 undervoltage clears RUN_LATCH even if USB keeps Pico alive; nominal10.333V, static screening9.75-10.94V. Shared fault line is not a separate input-voltage reading. | 1.8-5.5V comparator, OPEN-DRAIN, 1.242V reference; DBV SOT23-6" (at 340.36 219.71 0) (effects (font (size 1.0 1.0))  (hide yes)))
+(property "Description" "Post-eFuse VIN12 voltage monitor to Pico GP12 only; nominal10.333V, static screening9.75-10.94V. Does not clear RUN_LATCH or assert reset. | 1.8-5.5V comparator, OPEN-DRAIN, 1.242V reference; DBV SOT23-6" (at 340.36 219.71 0) (effects (font (size 1.0 1.0))  (hide yes)))
 (pin "3")
 (pin "4")
@@
 (global_label "VIN12_UV_REF" (shape passive) (at 363.22 209.55 0) (effects (font (size 1.0 1.0)) (justify left) ) (property "Intersheetrefs" "${INTERSHEET_REFS}" (at 363.22 209.55 0) (effects (font (size 0.8 0.8))  (hide yes))))
 (wire (pts (xy 358.14 219.71) (xy 363.22 219.71)) (stroke (width 0) (type default)))
-(global_label "HW_FAULT_N" (shape passive) (at 363.22 219.71 0) (effects (font (size 1.0 1.0)) (justify left) ) (property "Intersheetrefs" "${INTERSHEET_REFS}" (at 363.22 219.71 0) (effects (font (size 0.8 0.8))  (hide yes))))
+(global_label "VIN12_VALID" (shape passive) (at 363.22 219.71 0) (effects (font (size 1.0 1.0)) (justify left) ) (property "Intersheetrefs" "${INTERSHEET_REFS}" (at 363.22 219.71 0) (effects (font (size 0.8 0.8))  (hide yes))))
 (wire (pts (xy 358.14 199.39) (xy 363.22 199.39)) (stroke (width 0) (type default)))
 (global_label "3V3_CTRL" (shape passive) (at 363.22 199.39 0) (effects (font (size 1.0 1.0)) (justify left) ) (property "Intersheetrefs" "${INTERSHEET_REFS}" (at 363.22 199.39 0) (effects (font (size 0.8 0.8))  (hide yes))))
@@
 (wire (pts (xy 389.89 233.68) (xy 389.89 238.76)) (stroke (width 0) (type default)))
 (global_label "GND" (shape passive) (at 389.89 238.76 180) (effects (font (size 1.0 1.0)) (justify right) ) (property "Intersheetrefs" "${INTERSHEET_REFS}" (at 389.89 238.76 180) (effects (font (size 0.8 0.8))  (hide yes))))
-(text "U509: VIN12 loss clears RUN_LATCH. Nominal trip10.33V; qualify fast input interruptions with USB connected." (at 15 271 0) (effects (font (size 1.0 1.0)) (justify left top) ))
-(text "INA226 averaging window2.656ms: average rail telemetry only. No input-current ADC; bench supply reads total input." (at 15 278 0) (effects (font (size 1.0 1.0)) (justify left top) ))(sheet_instances (path "/f39c8d6a-e478-5a84-9c95-766dfa82ae02/396d387d-800b-5ee0-a374-8362af726b6a" (page "4"))) (embedded_fonts no))
+(text "U509: VIN12_VALID to Pico GP12, monitor-only; nominal threshold10.33V. Intrinsic UVLO or control brownout can still interrupt rails." (at 15 271 0) (effects (font (size 1.0 1.0)) (justify left top) ))
+(text "INA226 averaging window2.656ms: average rail telemetry only. No input-current ADC; bench supply reads total input." (at 15 278 0) (effects (font (size 1.0 1.0)) (justify left top) ))(sheet_instances (path "/f39c8d6a-e478-5a84-9c95-766dfa82ae02/396d387d-800b-5ee0-a374-8362af726b6a" (page "4"))) (embedded_fonts no)
+(symbol (lib_id "Sphinx_V2:Device__R") (at 281.94 245.11 0) (unit 1) (exclude_from_sim no) (in_bom yes) (on_board yes) (dnp no)
+(property "Reference" "R516" (at 285.94 243.86 0) (effects (font (size 1.0 1.0)) (justify left) ))
+(property "Value" "10k / 1%" (at 285.94 246.36 0) (effects (font (size 1.0 1.0)) (justify left) ))
+(property "Footprint" "Sphinx_V2:Resistor_SMD__R_0603_1608Metric" (at 281.94 245.11 0) (effects (font (size 1.0 1.0))  (hide yes)))
+(property "Datasheet" "https://yageogroup.com/component-documentation/download/specsheet/RC0603FR-0710KL" (at 281.94 245.11 0) (effects (font (size 1.0 1.0))  (hide yes)))
+(property "MPN" "RC0603FR-0710KL" (at 281.94 245.11 0) (effects (font (size 1.0 1.0))  (hide yes)))
+(property "Description" "Pullup for U509 VIN12_VALID monitor output to Pico GP12 | 10k +/-1% 0.1W 0603 thick film; +/-100ppm/C" (at 281.94 245.11 0) (effects (font (size 1.0 1.0))  (hide yes)))
+(pin "1")
+(pin "2")
+(instances (project "sphinx_power_v2" (path "/f39c8d6a-e478-5a84-9c95-766dfa82ae02/396d387d-800b-5ee0-a374-8362af726b6a" (reference "R516") (unit 1)))) )
+(wire (pts (xy 281.94 241.30) (xy 281.94 236.22)) (stroke (width 0) (type default)))
+(global_label "3V3_CTRL" (shape passive) (at 281.94 236.22 180) (effects (font (size 1.0 1.0)) (justify right)) (property "Intersheetrefs" "${INTERSHEET_REFS}" (at 281.94 236.22 180) (effects (font (size 0.8 0.8)) (hide yes))))
+(wire (pts (xy 281.94 248.92) (xy 281.94 254.00)) (stroke (width 0) (type default)))
+(global_label "VIN12_VALID" (shape passive) (at 281.94 254.00 180) (effects (font (size 1.0 1.0)) (justify right)) (property "Intersheetrefs" "${INTERSHEET_REFS}" (at 281.94 254.00 180) (effects (font (size 0.8 0.8)) (hide yes))))
+)

Commit message: Make V2 power state independent of Pico
Add an independently powered retained control domain, isolated I2C, hardware temperature and I/O overvoltage protection, and correct the socket keepout. Align operating requirements, BOM, schematic exports, and validation evidence.

Complete the final source review: zero ERC violations, 247 footprint/BOM matches, 80 ASIC pin checks, and 51 companion host tests including 122 interrupted-write cases. Record physical qualification limits and external companion firmware hashes.
Other:
- note added: "U509: VIN12_VALID to U903 P11, monitor-only; nominal threshold10.33V. Intrinsic UVLO or control brownout can still interrupt rails."
- note removed: "U509: VIN12_VALID to Pico GP12, monitor-only; nominal threshold10.33V. Intrinsic UVLO or control brownout can still interrupt rails."
Changed lines of the file:
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@@
 (kicad_sch (version 20250114) (generator "eeschema") (generator_version "10.0")
  (paper "A3")
-        (title_block (title "03 | Fixed 1.8 V I/O and calibrated telemetry") (date "2026-09-20") (rev "V2")
+        (title_block (title "03 | Fixed 1.8 V I/O and calibrated telemetry") (date "2026-09-22") (rev "V2")
         (company "Sphinx | Programmable power test board")
         (comment 1 "Review package: PCB, PI, SI, thermal and ASIC limits require qualification")
@@
 (property "Datasheet" "https://www.ti.com/lit/ds/symlink/tlv3011.pdf" (at 340.36 219.71 0) (effects (font (size 1.0 1.0))  (hide yes)))
 (property "MPN" "TLV3011AIDBVR" (at 340.36 219.71 0) (effects (font (size 1.0 1.0))  (hide yes)))
-(property "Description" "Post-eFuse VIN12 voltage monitor to Pico GP12 only; nominal10.333V, static screening9.75-10.94V. Does not clear RUN_LATCH or assert reset. | 1.8-5.5V comparator, OPEN-DRAIN, 1.242V reference; DBV SOT23-6" (at 340.36 219.71 0) (effects (font (size 1.0 1.0))  (hide yes)))
+(property "Description" "Post-eFuse VIN12 voltage monitor to U903 P11 only; nominal10.333V, static screening9.75-10.94V. Does not clear RUN_LATCH or assert reset. | 1.8-5.5V comparator, OPEN-DRAIN, 1.242V reference; DBV SOT23-6" (at 340.36 219.71 0) (effects (font (size 1.0 1.0))  (hide yes)))
 (pin "3")
 (pin "4")
@@
 (wire (pts (xy 389.89 233.68) (xy 389.89 238.76)) (stroke (width 0) (type default)))
 (global_label "GND" (shape passive) (at 389.89 238.76 180) (effects (font (size 1.0 1.0)) (justify right) ) (property "Intersheetrefs" "${INTERSHEET_REFS}" (at 389.89 238.76 180) (effects (font (size 0.8 0.8))  (hide yes))))
-(text "U509: VIN12_VALID to Pico GP12, monitor-only; nominal threshold10.33V. Intrinsic UVLO or control brownout can still interrupt rails." (at 15 271 0) (effects (font (size 1.0 1.0)) (justify left top) ))
+(text "U509: VIN12_VALID to U903 P11, monitor-only; nominal threshold10.33V. Intrinsic UVLO or control brownout can still interrupt rails." (at 15 271 0) (effects (font (size 1.0 1.0)) (justify left top) ))
 (text "INA226 averaging window2.656ms: average rail telemetry only. No input-current ADC; bench supply reads total input." (at 15 278 0) (effects (font (size 1.0 1.0)) (justify left top) ))(sheet_instances (path "/f39c8d6a-e478-5a84-9c95-766dfa82ae02/396d387d-800b-5ee0-a374-8362af726b6a" (page "4"))) (embedded_fonts no)
 (symbol (lib_id "Sphinx_V2:Device__R") (at 281.94 245.11 0) (unit 1) (exclude_from_sim no) (in_bom yes) (on_board yes) (dnp no)
@@
 (property "Datasheet" "https://yageogroup.com/component-documentation/download/specsheet/RC0603FR-0710KL" (at 281.94 245.11 0) (effects (font (size 1.0 1.0))  (hide yes)))
 (property "MPN" "RC0603FR-0710KL" (at 281.94 245.11 0) (effects (font (size 1.0 1.0))  (hide yes)))
-(property "Description" "Pullup for U509 VIN12_VALID monitor output to Pico GP12 | 10k +/-1% 0.1W 0603 thick film; +/-100ppm/C" (at 281.94 245.11 0) (effects (font (size 1.0 1.0))  (hide yes)))
-(pin "1")
-(pin "2")
+(property "Description" "Pullup for U509 VIN12_VALID monitor output to U903 P11 | 10k +/-1% 0.1W 0603 thick film; +/-100ppm/C" (at 281.94 245.11 0) (effects (font (size 1.0 1.0))  (hide yes)))
+(pin "1")
+(pin "2")
