File: schematic/04_usb_control.kicad_sch (KiCad schematic)
At the start: 14 parts, among them J401 PMBus debug (3.3V), J602 ZED REMOTE RESET, U401 Raspberry Pi Pico, U601 TLP293 GB

Commit message: Decouple DUT reset and input diagnostics from power interlocks
Use explicit manual, ZedBoard, and Pico reset requests. Route input-voltage validity to telemetry while retaining protective power interlocks. Synchronize requirements, schematic exports, BOM, and verification evidence.
Connections:
- net VIN12_VALID: now reaches U401.16 (GPIO12)
- net RESET_RELEASE renamed RESET_ASSERT
- no-connect marks 16 -> 15
Other:
- note added: "GP12 VIN12_VALID reports input validity only; no input voltage/current ADC."
- note added: "ON performs configuration and a single RUN_SET pulse. OFF and damage-risk faults clear RUN_LATCH; recovery needs ON. GP10 output: RUN_SET. GP5 input: RUN_LATCH. GP4 RESET_ASSERT: HIGH requests reset; LOW/high-Z releases."
- note added: "USB commands: SET / ON / OFF / RESET / STATUS. Hardware controls: STOP and DUT RESET; reset is explicit only."
- note removed: "No VIN/current telemetry: shared HW_FAULT_N indicates U509 input-low or another hardware fault."
- note removed: "ON performs configuration and a single RUN_SET pulse. OFF and faults clear the run latch; recovery needs a new ON. GP10 output: RUN_SET. GP5 input: RUN_LATCH. No manual ARM control or dedicated ARM indicators."
- note removed: "USB commands: SET / ON / OFF / STATUS. ON includes startup authorization. Hardware controls: STOP and DUT RESET."
Changed lines of the file:
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@@
 (kicad_sch (version 20250114) (generator "eeschema") (generator_version "10.0")
  (paper "A3")
-        (title_block (title "04 | USB control and remote reset") (date "2026-09-19") (rev "V2")
+        (title_block (title "04 | USB control and remote reset") (date "2026-09-20") (rev "V2")
         (company "Sphinx | Programmable power test board")
         (comment 1 "Review package: PCB, PI, SI, thermal and ASIC limits require qualification")
@@
         (comment 3 "Author: Yuchen Mei"))
         (text "Raspberry Pi Pico module: USB CDC + MicroPython controller; no proprietary USB/PMBus adapter required." (at 15 15 0) (effects (font (size 1.8 1.8)) (justify left top) ))
-(text "USB commands: SET / ON / OFF / STATUS. ON includes startup authorization. Hardware controls: STOP and DUT RESET." (at 15 23 0) (effects (font (size 1.27 1.27)) (justify left top) ))
+(text "USB commands: SET / ON / OFF / RESET / STATUS. Hardware controls: STOP and DUT RESET; reset is explicit only." (at 15 23 0) (effects (font (size 1.27 1.27)) (justify left top) ))
 (symbol (lib_id "Sphinx_V2:MCU_Module__RaspberryPi_Pico") (at 85.09 97.79 0) (unit 1) (exclude_from_sim no) (in_bom yes) (on_board yes) (dnp no)
 (property "Reference" "U401" (at 115.09 51.79 0) (effects (font (size 1.0 1.0)) (justify left) ))
@@
 (global_label "IO_REQ" (shape passive) (at 57.15 90.17 180) (effects (font (size 1.0 1.0)) (justify right) ) (property "Intersheetrefs" "${INTERSHEET_REFS}" (at 57.15 90.17 180) (effects (font (size 0.8 0.8))  (hide yes))))
 (wire (pts (xy 62.23 92.71) (xy 57.15 92.71)) (stroke (width 0) (type default)))
-(global_label "RESET_RELEASE" (shape passive) (at 57.15 92.71 180) (effects (font (size 1.0 1.0)) (justify right) ) (property "Intersheetrefs" "${INTERSHEET_REFS}" (at 57.15 92.71 180) (effects (font (size 0.8 0.8))  (hide yes))))
+(global_label "RESET_ASSERT" (shape passive) (at 57.15 92.71 180) (effects (font (size 1.0 1.0)) (justify right) ) (property "Intersheetrefs" "${INTERSHEET_REFS}" (at 57.15 92.71 180) (effects (font (size 0.8 0.8))  (hide yes))))
 (wire (pts (xy 62.23 95.25) (xy 57.15 95.25)) (stroke (width 0) (type default)))
 (global_label "RUN_LATCH" (shape passive) (at 57.15 95.25 180) (effects (font (size 1.0 1.0)) (justify right) ) (property "Intersheetrefs" "${INTERSHEET_REFS}" (at 57.15 95.25 180) (effects (font (size 0.8 0.8))  (hide yes))))
@@
 (wire (pts (xy 62.23 110.49) (xy 57.15 110.49)) (stroke (width 0) (type default)))
 (global_label "MON_ALERT_N" (shape passive) (at 57.15 110.49 180) (effects (font (size 1.0 1.0)) (justify right) ) (property "Intersheetrefs" "${INTERSHEET_REFS}" (at 57.15 110.49 180) (effects (font (size 0.8 0.8))  (hide yes))))
-(no_connect (at 62.23 113.03))
 (no_connect (at 62.23 115.57))
 (no_connect (at 62.23 118.11))
@@
 (global_label "GND" (shape passive) (at 355.6 243.84 180) (effects (font (size 1.0 1.0)) (justify right) ) (property "Intersheetrefs" "${INTERSHEET_REFS}" (at 355.6 243.84 180) (effects (font (size 0.8 0.8))  (hide yes))))
 (text "USB host controls the sweep. Pico implements output sequencing, fault handling, and watchdog.\n19 points: 0.30-1.20V / 0.05V steps. Scale changes perform a controlled power-cycle.\nJ401 exposes only the debug bus; it does not replace the Pico safety state machine.\nAUX5V keeps control power independent of the PC connection." (at 25 196 0) (effects (font (size 1.1 1.1)) (justify left top) ))
-(text "No VIN/current telemetry: shared HW_FAULT_N indicates U509 input-low or another hardware fault." (at 150 268 0) (effects (font (size 0.95 0.95)) (justify left top) ))
+(text "GP12 VIN12_VALID reports input validity only; no input voltage/current ADC." (at 150 268 0) (effects (font (size 0.95 0.95)) (justify left top) ))
 (symbol (lib_id "Sphinx_V2:Device__R") (at 129.54 153.67 0) (unit 1) (exclude_from_sim no) (in_bom yes) (on_board yes) (dnp no)
 (property "Reference" "R411" (at 133.54 152.42 0) (effects (font (size 1.0 1.0)) (justify left) ))
@@
 (property "Datasheet" "https://yageogroup.com/component-documentation/download/specsheet/RC0603FR-07100KL" (at 129.54 153.67 0) (effects (font (size 1.0 1.0))  (hide yes)))
 (property "MPN" "RC0603FR-07100KL" (at 129.54 153.67 0) (effects (font (size 1.0 1.0))  (hide yes)))
-(property "Description" "100k +/-1% 0.1W 0603 thick film; +/-100ppm/C" (at 129.54 153.67 0) (effects (font (size 1.0 1.0))  (hide yes)))
+(property "Description" "Pico RESET_ASSERT gate pulldown; place next to Q602 to keep reset request inactive with GPIO unpowered or high-Z | 100k +/-1% 0.1W 0603 thick film; +/-100ppm/C" (at 129.54 153.67 0) (effects (font (size 1.0 1.0))  (hide yes)))
 (pin "1")
 (pin "2")
 (instances (project "sphinx_power_v2" (path "/f39c8d6a-e478-5a84-9c95-766dfa82ae02/75c9142f-37c4-500b-ad86-039aa4577f35" (reference "R411") (unit 1)))) )
 (wire (pts (xy 129.54 149.86) (xy 129.54 144.78)) (stroke (width 0) (type default)))
-(global_label "RESET_RELEASE" (shape passive) (at 129.54 144.78 180) (effects (font (size 1.0 1.0)) (justify right) ) (property "Intersheetrefs" "${INTERSHEET_REFS}" (at 129.54 144.78 180) (effects (font (size 0.8 0.8))  (hide yes))))
+(global_label "RESET_ASSERT" (shape passive) (at 129.54 144.78 180) (effects (font (size 1.0 1.0)) (justify right) ) (property "Intersheetrefs" "${INTERSHEET_REFS}" (at 129.54 144.78 180) (effects (font (size 0.8 0.8))  (hide yes))))
 (wire (pts (xy 129.54 157.48) (xy 129.54 162.56)) (stroke (width 0) (type default)))
 (global_label "GND" (shape passive) (at 129.54 162.56 180) (effects (font (size 1.0 1.0)) (justify right) ) (property "Intersheetrefs" "${INTERSHEET_REFS}" (at 129.54 162.56 180) (effects (font (size 0.8 0.8))  (hide yes))))
@@
 (wire (pts (xy 62.23 107.95) (xy 57.15 107.95)) (stroke (width 0) (type default)))
 (global_label "RUN_SET" (shape passive) (at 57.15 107.95 180) (effects (font (size 1.0 1.0)) (justify right) ) (property "Intersheetrefs" "${INTERSHEET_REFS}" (at 57.15 107.95 180) (effects (font (size 0.8 0.8))  (hide yes))))
-(text "ON performs configuration and a single RUN_SET pulse.\nOFF and faults clear the run latch; recovery needs a new ON.\nGP10 output: RUN_SET. GP5 input: RUN_LATCH.\nNo manual ARM control or dedicated ARM indicators." (at 160 147 0) (effects (font (size 1.1 1.1)) (justify left top) )))
+(text "ON performs configuration and a single RUN_SET pulse.\nOFF and damage-risk faults clear RUN_LATCH; recovery needs ON.\nGP10 output: RUN_SET. GP5 input: RUN_LATCH.\nGP4 RESET_ASSERT: HIGH requests reset; LOW/high-Z releases." (at 160 147 0) (effects (font (size 1.1 1.1)) (justify left top) ))
+(wire (pts (xy 62.23 113.03) (xy 57.15 113.03)) (stroke (width 0) (type default)))
+(global_label "VIN12_VALID" (shape passive) (at 57.15 113.03 180) (effects (font (size 1.0 1.0)) (justify right)) (property "Intersheetrefs" "${INTERSHEET_REFS}" (at 57.15 113.03 180) (effects (font (size 0.8 0.8)) (hide yes))))
+)

Commit message: Make V2 power state independent of Pico
Add an independently powered retained control domain, isolated I2C, hardware temperature and I/O overvoltage protection, and correct the socket keepout. Align operating requirements, BOM, schematic exports, and validation evidence.

Complete the final source review: zero ERC violations, 247 footprint/BOM matches, 80 ASIC pin checks, and 51 companion host tests including 122 interrupted-write cases. Record physical qualification limits and external companion firmware hashes.
Connections:
- net 3V3_CTRL: no longer U401.36 (3V3)
- net BOARD_NTC: no longer U401.32 (GPIO27_ADC1)
- net CORE_ALERT_N: no longer U401.12 (GPIO9)
- net MON_ALERT_N: no longer U401.15 (GPIO11)
- net PMBUS_SCL: no longer U401.2 (GPIO1)
- net PMBUS_SDA: no longer U401.1 (GPIO0)
- net RESET_ASSERT: no longer U401.6 (GPIO4)
- net CORE_PG: no longer names the net of U401.9 (GPIO6)
- net CORE_REQ: no longer names the net of U401.4 (GPIO2)
- net HW_FAULT_N: no longer names the net of U401.11 (GPIO8)
- net HW_FAULT_N: no longer U401.20 (GPIO15)
- net IO_REQ: no longer names the net of U401.5 (GPIO3)
- net IO_VALID: no longer names the net of U401.10 (GPIO7)
- net RUN_LATCH: no longer names the net of U401.7 (GPIO5)
- net RUN_SET: no longer names the net of U401.14 (GPIO10)
- net VIN12_VALID: no longer names the net of U401.16 (GPIO12)
- new net PICO_3V3: U401.36 (3V3)
- new net PICO_SCL: U401.2 (GPIO1)
- new net PICO_SDA: U401.1 (GPIO0)
- no-connect marks 15 -> 28
Other:
- note added: "All Pico GPIOs except GP0/GP1 are unconnected. GPIO expander U903 drives RUN_SET, CORE_REQ, IO_REQ and held RESET_ASSERT. Q901 provides fault clear. Explicit OFF and physical STOP remain available."
- note added: "Pico is a command-only USB interface. Board state and protection are independent. I2C is isolated by U902; U903 retains CORE / IO / RESET requests. Pico boot, USB inactivity and communication errors do not change outputs. See sheets09/10 and docs/AUTONOMOUS_POWER.md."
- note removed: "GP12 VIN12_VALID reports input validity only; no input voltage/current ADC."
- note removed: "GP15: OPEN-DRAIN shutdown; LOW clears RUN_LATCH. Never drive HW_FAULT_N push-pull HIGH."
- note removed: "ON performs configuration and a single RUN_SET pulse. OFF and damage-risk faults clear RUN_LATCH; recovery needs ON. GP10 output: RUN_SET. GP5 input: RUN_LATCH. GP4 RESET_ASSERT: HIGH requests reset; LOW/high-Z releases."
- note removed: "USB host controls the sweep. Pico implements output sequencing, fault handling, and watchdog. 19 points: 0.30-1.20V / 0.05V steps. Scale changes perform a controlled power-cycle. J401 exposes only the debug bus; it does not replace the Pico safety state machine. AUX5V keeps control power independent of the PC connection."
