File: schematic/05_hardware_safety.kicad_sch (KiCad schematic)
At the start: 19 parts, among them SW502 STOP, U501 TLV3011AIDBVR, U502 TPS3808G33DBVR, U503 SN74LVC1G74DCUR, U504 74LVC08AT14-13, U506 SN74LVC1G11DCKR, U507 SN74LVC2G17DBVT

Commit message: Decouple DUT reset and input diagnostics from power interlocks
Use explicit manual, ZedBoard, and Pico reset requests. Route input-voltage validity to telemetry while retaining protective power interlocks. Synchronize requirements, schematic exports, BOM, and verification evidence.
Parts:
- removed C507: 100n / 16V, Sphinx_V2:Capacitor_SMD__C_0402_1005Metric, symbol Sphinx_V2:Device__C
- removed U506: SN74LVC1G11DCKR, Sphinx_V2:Package_TO_SOT_SMD__SOT-363_SC-70-6, symbol Sphinx_V2:74xGxx__74LVC1G11
Connections:
- net RESET_RELEASE is gone; now on net GND: U504.10 (3B)
- net GND: now also U504.9 (3A)
- net RUN_LATCH: no longer U504.9 (3A)
- net RESET_PERMIT: no longer names the net of U504.8 (3Y)
- no-connect marks 3 -> 4
Other:
- note added: "C502-U501; C503-U502; C504-U503. C506-U504; C508-U507. Place each bypass capacitor at its IC."
- note added: "Core OVP and eFuse FLT retain hardware shutdown. VIN12_VALID, CORE_PG and IO_VALID are monitor-only."
- note added: "DUT reset is independent of RUN_LATCH and PG. At valid 1.8V, reset defaults LOW (released). Only SW601, U601 or Pico RESET_ASSERT assert reset."
- note added: "ON sets the run latch. STOP, damage-risk faults or control brownout clear it; recovery requires a new ON command."
- note removed: "C502-U501; C503-U502; C504-U503. C506-U504; C507-U506; C508-U507. Place each bypass capacitor at its IC."
- note removed: "No manual ARM step. Core OVP, VIN12 loss, eFuse fault and control brownout still shut down both rails in hardware."
- note removed: "ON sets the run latch automatically. STOP or a hardware fault clears it; recovery requires a new ON command."
- title: 05 | Fault shutdown latch and power-qualified reset -> 05 | Hardware power shutdown latch

Commit message: Make V2 power state independent of Pico
Add an independently powered retained control domain, isolated I2C, hardware temperature and I/O overvoltage protection, and correct the socket keepout. Align operating requirements, BOM, schematic exports, and validation evidence.

Complete the final source review: zero ERC violations, 247 footprint/BOM matches, 80 ASIC pin checks, and 51 companion host tests including 122 interrupted-write cases. Record physical qualification limits and external companion firmware hashes.
Connections:
- net SUPERVISOR_CT: now reaches U502.4 (CT)
- no-connect marks 4 -> 3
Other:
- note added: "DUT reset is independent of RUN_LATCH and PG. At valid 1.8V, reset defaults LOW (released). Only SW601, U601 or U903 RESET_ASSERT assert reset."
- note added: "U903 P03: one RUN_SET pulse inside ON, after configuration. U903 P04 / Q901: LOW / high impedance only on HW_FAULT_N. A stuck-high RUN_SET cannot restart a cleared latch."
- note removed: "DUT reset is independent of RUN_LATCH and PG. At valid 1.8V, reset defaults LOW (released). Only SW601, U601 or Pico RESET_ASSERT assert reset."
- note removed: "GP10: one RUN_SET pulse inside ON, after configuration. GP15: LOW / high impedance only on HW_FAULT_N. A stuck-high RUN_SET cannot restart a cleared latch."
Changed lines of the file:
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@@
 (kicad_sch (version 20250114) (generator "eeschema") (generator_version "10.0")
  (paper "A3")
-        (title_block (title "05 | Hardware power shutdown latch") (date "2026-09-20") (rev "V2")
+        (title_block (title "05 | Hardware power shutdown latch") (date "2026-09-22") (rev "V2")
         (company "Sphinx | Programmable power test board")
         (comment 1 "Review package: PCB, PI, SI, thermal and ASIC limits require qualification")
@@
 (property "Datasheet" "https://www.ti.com/lit/ds/symlink/tps3808.pdf" (at 204.47 69.85 0) (effects (font (size 1.0 1.0))  (hide yes)))
 (property "MPN" "TPS3808G33DBVR" (at 204.47 69.85 0) (effects (font (size 1.0 1.0))  (hide yes)))
-(property "Description" "Control-supply supervisor; CT open gives approximately 20 ms startup reset, threshold 3.07 V. | 0.9-6.5V supervisor, G33 threshold3.07V, open-drain reset, CT open approx20ms; DBV6" (at 204.47 69.85 0) (effects (font (size 1.0 1.0))  (hide yes)))
+(property "Description" "Control-supply supervisor; CT100k pullup gives180-420ms startup reset, threshold 3.07 V. | 0.9-6.5V supervisor, G33 threshold3.07V, open-drain reset, CT100k pullup:180-420ms (300ms nominal); DBV6" (at 204.47 69.85 0) (effects (font (size 1.0 1.0))  (hide yes)))
 (pin "5")
 (pin "3")
@@
 (wire (pts (xy 186.69 69.85) (xy 181.61 69.85)) (stroke (width 0) (type default)))
 (global_label "3V3_CTRL" (shape passive) (at 181.61 69.85 180) (effects (font (size 1.0 1.0)) (justify right) ) (property "Intersheetrefs" "${INTERSHEET_REFS}" (at 181.61 69.85 180) (effects (font (size 0.8 0.8))  (hide yes))))
-(no_connect (at 186.69 80.01))
 (wire (pts (xy 222.25 59.69) (xy 227.33 59.69)) (stroke (width 0) (type default)))
 (global_label "3V3_CTRL" (shape passive) (at 227.33 59.69 0) (effects (font (size 1.0 1.0)) (justify left) ) (property "Intersheetrefs" "${INTERSHEET_REFS}" (at 227.33 59.69 0) (effects (font (size 0.8 0.8))  (hide yes))))
@@
 (property "Datasheet" "https://yageogroup.com/component-documentation/download/specsheet/RC0603FR-0710KL" (at 330.2 128.27 0) (effects (font (size 1.0 1.0))  (hide yes)))
 (property "MPN" "RC0603FR-0710KL" (at 330.2 128.27 0) (effects (font (size 1.0 1.0))  (hide yes)))
-(property "Description" "Holds run-latch clock low while Pico GP10 is high impedance. | 10k +/-1% 0.1W 0603 thick film; +/-100ppm/C" (at 330.2 128.27 0) (effects (font (size 1.0 1.0))  (hide yes)))
+(property "Description" "Holds run-latch clock low while U903 P03 is high impedance. | 10k +/-1% 0.1W 0603 thick film; +/-100ppm/C" (at 330.2 128.27 0) (effects (font (size 1.0 1.0))  (hide yes)))
 (pin "1")
 (pin "2")
@@
 (wire (pts (xy 335.28 173.99) (xy 340.36 173.99)) (stroke (width 0) (type default)))
 (global_label "GND" (shape passive) (at 340.36 173.99 0) (effects (font (size 1.0 1.0)) (justify left) ) (property "Intersheetrefs" "${INTERSHEET_REFS}" (at 340.36 173.99 0) (effects (font (size 0.8 0.8))  (hide yes))))
-(text "GP10: one RUN_SET pulse inside ON, after configuration.\nGP15: LOW / high impedance only on HW_FAULT_N.\nA stuck-high RUN_SET cannot restart a cleared latch." (at 245 190 0) (effects (font (size 0.95 0.95)) (justify left top) ))
+(text "U903 P03: one RUN_SET pulse inside ON, after configuration.\nU903 P04 / Q901: LOW / high impedance only on HW_FAULT_N.\nA stuck-high RUN_SET cannot restart a cleared latch." (at 245 190 0) (effects (font (size 0.95 0.95)) (justify left top) ))
 (symbol (lib_id "Sphinx_V2:74LVC08A_TSSOP14") (at 91.44 213.36 0) (unit 1) (exclude_from_sim no) (in_bom yes) (on_board yes) (dnp no)
 (property "Reference" "U504" (at 91.44 174.34 0) (effects (font (size 1.0 1.0))  ))
@@
 (text "C502-U501; C503-U502; C504-U503.\nC506-U504; C508-U507.\nPlace each bypass capacitor at its IC." (at 215 250 0) (effects (font (size 0.9 0.9)) (justify left top) ))(sheet_instances (path "/f39c8d6a-e478-5a84-9c95-766dfa82ae02/95ce739b-4eee-5f42-a669-179a7d0060de" (page "6"))) (embedded_fonts no)
 (no_connect (at 114.3 220.98))
-(text "DUT reset is independent of RUN_LATCH and PG.\nAt valid 1.8V, reset defaults LOW (released).\nOnly SW601, U601 or Pico RESET_ASSERT assert reset." (at 210 208 0) (effects (font (size 1.0 1.0)) (justify left top)))
+(text "DUT reset is independent of RUN_LATCH and PG.\nAt valid 1.8V, reset defaults LOW (released).\nOnly SW601, U601 or U903 RESET_ASSERT assert reset." (at 210 208 0) (effects (font (size 1.0 1.0)) (justify left top)))
+(wire (pts (xy 186.69 80.01) (xy 181.61 80.01)) (stroke (width 0) (type default)))
+(global_label "SUPERVISOR_CT" (shape passive) (at 181.61 80.01 180) (effects (font (size 1 1)) (justify right)) (property "Intersheetrefs" "${INTERSHEET_REFS}" (at 181.61 80.01 180) (effects (font (size 0.8 0.8)) (hide yes))))
 )
