File: schematic/08_io_decoupling.kicad_sch (KiCad schematic)
At the start: 27 parts, among them U508 TLV3011AIDBVR

Commit message: Decouple DUT reset and input diagnostics from power interlocks
Use explicit manual, ZedBoard, and Pico reset requests. Route input-voltage validity to telemetry while retaining protective power interlocks. Synchronize requirements, schematic exports, BOM, and verification evidence.
Other:
- note added: "IO_VALID threshold nominal1.626V; conservative static bounds about1.56-1.70V. Monitor-only; no reset or latching UV cutoff."
- note added: "U508 measures VIO directly. IO_VALID reports to Pico GP7 only; regulator IO_PG is only used by FSW."
- note removed: "IO_VALID trip nominal1.626V; conservative static bounds about1.56-1.70V. Hardware reset qualifier, not a latching UV cutoff."
- note removed: "U508 measures VIO directly. IO_VALID qualifies RESET and Pico GP7; regulator IO_PG is only used by FSW."
- title: 08 | I/O decoupling and undervoltage reset interlock -> 08 | I/O decoupling and voltage monitor
Changed lines of the file:
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@@
 (kicad_sch (version 20250114) (generator "eeschema") (generator_version "10.0")
  (paper "A3")
-        (title_block (title "08 | I/O decoupling and undervoltage reset interlock") (date "2026-09-19") (rev "V2")
+        (title_block (title "08 | I/O decoupling and voltage monitor") (date "2026-09-20") (rev "V2")
         (company "Sphinx | Programmable power test board")
         (comment 1 "Review package: PCB, PI, SI, thermal and ASIC limits require qualification")
@@
         (comment 3 "Author: Yuchen Mei"))
         (text "Fixed1.8V I/O supply: distributed local decoupling. Scope connections are high impedance." (at 15 15 0) (effects (font (size 1.8 1.8)) (justify left top) ))
-(text "U508 measures VIO directly. IO_VALID qualifies RESET and Pico GP7; regulator IO_PG is only used by FSW." (at 15 23 0) (effects (font (size 1.1 1.1)) (justify left top) ))
+(text "U508 measures VIO directly. IO_VALID reports to Pico GP7 only; regulator IO_PG is only used by FSW." (at 15 23 0) (effects (font (size 1.1 1.1)) (justify left top) ))
 (symbol (lib_id "Sphinx_V2:Device__C") (at 35.56 58.42 0) (unit 1) (exclude_from_sim no) (in_bom yes) (on_board yes) (dnp no)
 (property "Reference" "C801" (at 39.56 57.17 0) (effects (font (size 1.0 1.0)) (justify left) ))
@@
 (property "Datasheet" "https://www.ti.com/lit/ds/symlink/tlv3011.pdf" (at 72.39 229.87 0) (effects (font (size 1.0 1.0))  (hide yes)))
 (property "MPN" "TLV3011AIDBVR" (at 72.39 229.87 0) (effects (font (size 1.0 1.0))  (hide yes)))
-(property "Description" "Independent VIO undervoltage qualifier, nominal1.626V; coarse backup, not ASIC rated threshold | 1.8-5.5V comparator, OPEN-DRAIN, 1.242V reference; DBV SOT23-6" (at 72.39 229.87 0) (effects (font (size 1.0 1.0))  (hide yes)))
+(property "Description" "Independent VIO monitor to Pico GP7 only, nominal1.626V; no reset or hardware shutdown action | 1.8-5.5V comparator, OPEN-DRAIN, 1.242V reference; DBV SOT23-6" (at 72.39 229.87 0) (effects (font (size 1.0 1.0))  (hide yes)))
 (pin "3")
 (pin "4")
@@
 (wire (pts (xy 292.1 232.41) (xy 292.1 237.49)) (stroke (width 0) (type default)))
 (global_label "IO_VALID" (shape passive) (at 292.1 237.49 180) (effects (font (size 1.0 1.0)) (justify right) ) (property "Intersheetrefs" "${INTERSHEET_REFS}" (at 292.1 237.49 180) (effects (font (size 0.8 0.8))  (hide yes))))
-(text "IO_VALID trip nominal1.626V; conservative static bounds about1.56-1.70V. Hardware reset qualifier, not a latching UV cutoff." (at 15 266 0) (effects (font (size 1.0 1.0)) (justify left top) ))
+(text "IO_VALID threshold nominal1.626V; conservative static bounds about1.56-1.70V. Monitor-only; no reset or latching UV cutoff." (at 15 266 0) (effects (font (size 1.0 1.0)) (justify left top) ))
 (text "Place U508 divider at socket VIO; decouple each IC locally. Adjacent GND probe pads; high-Z probing; continuous signal return plane." (at 15 274 0) (effects (font (size 1.0 1.0)) (justify left top) ))(sheet_instances (path "/f39c8d6a-e478-5a84-9c95-766dfa82ae02/36761b75-2b3e-5b16-bc66-e4b7245270a9" (page "9"))) (embedded_fonts no))

Commit message: Make V2 power state independent of Pico
Add an independently powered retained control domain, isolated I2C, hardware temperature and I/O overvoltage protection, and correct the socket keepout. Align operating requirements, BOM, schematic exports, and validation evidence.

Complete the final source review: zero ERC violations, 247 footprint/BOM matches, 80 ASIC pin checks, and 51 companion host tests including 122 interrupted-write cases. Record physical qualification limits and external companion firmware hashes.
Other:
- note added: "U508 measures VIO directly. IO_VALID reports to U903 P10 only; regulator IO_PG is only used by FSW."
- note removed: "U508 measures VIO directly. IO_VALID reports to Pico GP7 only; regulator IO_PG is only used by FSW."
Changed lines of the file:
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@@
 (kicad_sch (version 20250114) (generator "eeschema") (generator_version "10.0")
  (paper "A3")
-        (title_block (title "08 | I/O decoupling and voltage monitor") (date "2026-09-20") (rev "V2")
+        (title_block (title "08 | I/O decoupling and voltage monitor") (date "2026-09-22") (rev "V2")
         (company "Sphinx | Programmable power test board")
         (comment 1 "Review package: PCB, PI, SI, thermal and ASIC limits require qualification")
@@
         (comment 3 "Author: Yuchen Mei"))
         (text "Fixed1.8V I/O supply: distributed local decoupling. Scope connections are high impedance." (at 15 15 0) (effects (font (size 1.8 1.8)) (justify left top) ))
-(text "U508 measures VIO directly. IO_VALID reports to Pico GP7 only; regulator IO_PG is only used by FSW." (at 15 23 0) (effects (font (size 1.1 1.1)) (justify left top) ))
+(text "U508 measures VIO directly. IO_VALID reports to U903 P10 only; regulator IO_PG is only used by FSW." (at 15 23 0) (effects (font (size 1.1 1.1)) (justify left top) ))
 (symbol (lib_id "Sphinx_V2:Device__C") (at 35.56 58.42 0) (unit 1) (exclude_from_sim no) (in_bom yes) (on_board yes) (dnp no)
 (property "Reference" "C801" (at 39.56 57.17 0) (effects (font (size 1.0 1.0)) (justify left) ))
@@
 (property "Datasheet" "https://www.ti.com/lit/ds/symlink/tlv3011.pdf" (at 72.39 229.87 0) (effects (font (size 1.0 1.0))  (hide yes)))
 (property "MPN" "TLV3011AIDBVR" (at 72.39 229.87 0) (effects (font (size 1.0 1.0))  (hide yes)))
-(property "Description" "Independent VIO monitor to Pico GP7 only, nominal1.626V; no reset or hardware shutdown action | 1.8-5.5V comparator, OPEN-DRAIN, 1.242V reference; DBV SOT23-6" (at 72.39 229.87 0) (effects (font (size 1.0 1.0))  (hide yes)))
+(property "Description" "Independent VIO monitor to U903 P10 only, nominal1.626V; no reset or hardware shutdown action | 1.8-5.5V comparator, OPEN-DRAIN, 1.242V reference; DBV SOT23-6" (at 72.39 229.87 0) (effects (font (size 1.0 1.0))  (hide yes)))
 (pin "3")
 (pin "4")
